Commit message: V0.2.1 New URDF

File: URDF/mppi/urdf/mppi.urdf (robot description, URDF)
Before this commit: robot mppi, 3 links, 2 joints
Links:
- link Link_1: mass 0.0688716456981545 -> 0.067836
- link Link_2: mass 0.00521037344424208 -> 0.031109
- link base_link: mass 0.130648831366131 -> 1.1619
Joints:
- joint Joint_1: limit (none) -> lower=-0.8 upper=0.8 effort=0 velocity=0; origin xyz=0 -0.0735 -0.000250000000000003 rpy=-1.5707963267949 0 0 -> xyz=0.076125 -0.042332 -0.059398 rpy=-0.0039907 0 0
- joint Joint_2: limit (none) -> lower=-0.8 upper=0.8 effort=0 velocity=0; origin xyz=0 0 -0.1608 rpy=3.14159265358979 0 0 -> xyz=0 0 -0.1308 rpy=3.1379 0 0
