Commit message: V0.4.2 Centered  and orientated model

File: SkyGrip_URDF/urdf/SkyGrip_URDF.urdf (robot description, URDF)
Before this commit: robot SkyGrip_URDF, 3 links, 2 joints
Joints:
- joint Joint_1: origin xyz=0.075884 -0.042123 -0.023898 rpy=-0.00065513 0 -0.0087266 -> xyz=0 -2.5E-05 -0.038 rpy=-0.00065513 0 0
